File: ASD2004.brd (EAGLE design)
At the start: 22.5 x 22.5 mm, 23 parts, among them J1 PIN_1X.1"1, J10 PIN_1X.1"1, J11 PIN_1X.1"1, J12 DF12-32-DS, J13 PIN_1X.1"1, J14 PIN_1X.1"1, J15 PIN_1X.1"1, J16 PIN_1X.1"1, J17 PIN_1X.1"1, J18 PIN_1X.1"1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

Commit message: Updated to Rev 2
Routing:
- net AREF: track 6.88 -> 0.00 mm, vias 1 -> 0
- net VBATT: track 30.2 -> 29.2 mm, vias 0 -> 2
Other:
- board text added: "0"
- board text added: "2"
- board text added: "3"
- board text added: "4"
- board text added: "5"
- board text added: "6"
- board text added: "7"
- board text added: "8"
- board text added: "9"
- board text added: "A4"
- board text added: "A5"
- board text added: "REV 2"
- board text removed: "IO0"
- board text removed: "IO1"
- board text removed: "IO2"
- board text removed: "IO3"
- board text removed: "IO4"
- board text removed: "IO5"
- board text removed: "IO6"
- board text removed: "IO7"
- board text removed: "IO8"
- board text removed: "IO9"
- board text removed: "REV 1"
- board text removed: "SCL"
- board text removed: "SDA"
